File: ProyFinalMateriales/ProyFinalMateriales.kicad_pcb (KiCad board)
At the start: 2 copper layers, 48 x 67.9 mm, 12 parts, among them U1 NodeMCU1.0(ESP-12E)

Commit message: update
Routing:
- net 5V: track 74.5 -> 67.2 mm
- net GND1: track 177.1 -> 176.2 mm
Other:
- board text added: "CANSAT"
Changed lines of the file:
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@@
       (svguseinch false)
       (svgprecision 6)
-      (excludeedgelayer true)
+      (excludeedgelayer false)
       (plotframeref false)
       (viasonmask false)
@@
       (drillshape 0)
       (scaleselection 1)
-      (outputdirectory "C:/Users/Camilo/OneDrive - Universidad de los Andes/6Sexto Semestre (2022-2)/Materiales IEE/ProyFinal/ArchivosPCB/")
+      (outputdirectory "../../../OneDrive - Universidad de los Andes/6Sexto Semestre (2022-2)/Materiales IEE/ProyFinal/ArchivosPCB/")
     )
   )
@@
   )
   (gr_rect (start 100 135.5) (end 148 67.56) (layer "Edge.Cuts") (width 0.1) (fill none))
+  (gr_text "CANSAT" (at 137.16 109.22) (layer "F.Cu")
+    (effects (font (size 1.5 1.5) (thickness 0.3)))
+  )
   (gr_text "Proy. Final\nMateriales para IEE\nCamilo Morillo\nAlejandro Salaz" (at 136.7 108.7) (layer "B.Cu")
     (effects (font (size 1 1) (thickness 0.2)) (justify mirror))
@@
   (segment (start 108.5 122.765) (end 106.69 122.765) (width 0.3) (layer "B.Cu") (net 2))
   (segment (start 141.475 92.475) (end 131.5 92.475) (width 0.3) (layer "B.Cu") (net 3))
-  (segment (start 145.5 83.765) (end 143.5 81.765) (width 0.3) (layer "B.Cu") (net 3))
+  (segment (start 143.51 120.65) (end 143.11 120.65) (width 0.3) (layer "B.Cu") (net 3))
   (segment (start 141.5 92.5) (end 141.475 92.475) (width 0.3) (layer "B.Cu") (net 3))
+  (segment (start 143.5 88.91) (end 143.5 90.5) (width 0.3) (layer "B.Cu") (net 3))
+  (segment (start 144.78 119.38) (end 143.51 120.65) (width 0.3) (layer "B.Cu") (net 3))
   (segment (start 143 120.54) (end 139.92 123.62) (width 0.3) (layer "B.Cu") (net 3))
   (segment (start 143.5 90.5) (end 141.5 92.5) (width 0.3) (layer "B.Cu") (net 3))
-  (segment (start 143.5 81.765) (end 143.5 90.5) (width 0.3) (layer "B.Cu") (net 3))
-  (segment (start 145.5 118.04) (end 145.5 83.765) (width 0.3) (layer "B.Cu") (net 3))
+  (segment (start 143.5 81.765) (end 143.5 88.91) (width 0.3) (layer "B.Cu") (net 3))
+  (segment (start 144.78 90.19) (end 144.78 119.38) (width 0.3) (layer "B.Cu") (net 3))
+  (segment (start 143.5 88.91) (end 144.78 90.19) (width 0.3) (layer "B.Cu") (net 3))
+  (segment (start 143.11 120.65) (end 143 120.54) (width 0.3) (layer "B.Cu") (net 3))
   (segment (start 139.92 123.62) (end 132 123.62) (width 0.3) (layer "B.Cu") (net 3))
-  (segment (start 143 120.54) (end 145.5 118.04) (width 0.3) (layer "B.Cu") (net 3))
   (segment (start 108.5 81.265) (end 108.5 85.5) (width 0.3) (layer "F.Cu") (net 4))
   (segment (start 119.535 107.665) (end 124.7 102.5) (width 0.3) (layer "F.Cu") (net 4))
   (segment (start 136.8 118) (end 134.8 116) (width 0.3) (layer "F.Cu") (net 4))
   (segment (start 134.4 95.5) (end 133.9 95) (width 0.3) (layer "F.Cu") (net 4))
-  (segment (start 103.9 122) (end 101.8 122) (width 0.3) (layer "F.Cu") (net 4))
-  (segment (start 101.3 81.6) (end 101.635 81.265) (width 0.3) (layer "F.Cu") (net 4))
   (segment (start 134.8 116) (end 132 116) (width 0.3) (layer "F.Cu") (net 4))
-  (segment (start 105.7 107.9) (end 104.7 108.9) (width 0.3) (layer "F.Cu") (net 4))
+  (segment (start 101.3 121.5) (end 101.3 83.01) (width 0.3) (layer "F.Cu") (net 4))
   (segment (start 117.5 107.665) (end 119.535 107.665) (width 0.3) (layer "F.Cu") (net 4))
   (segment (start 119.7 126.3) (end 115.3 126.3) (width 0.3) (layer "F.Cu") (net 4))
   (segment (start 108.5 85.5) (end 106.4 87.6) (width 0.3) (layer "F.Cu") (net 4))
+  (segment (start 101.8 122) (end 101.3 121.5) (width 0.3) (layer "F.Cu") (net 4))
   (segment (start 116.135 107.665) (end 117.5 107.665) (width 0.3) (layer "F.Cu") (net 4))
   (segment (start 121 125) (end 119.7 126.3) (width 0.3) (layer "F.Cu") (net 4))
   (segment (start 143 118) (end 136.8 118) (width 0.3) (layer "F.Cu") (net 4))
+  (segment (start 103.9 122) (end 101.8 122) (width 0.3) (layer "F.Cu") (net 4))
   (segment (start 115.3 126.3) (end 114.3 125.3) (width 0.3) (layer "F.Cu") (net 4))
-  (segment (start 101.3 121.5) (end 101.3 81.6) (width 0.3) (layer "F.Cu") (net 4))
-  (segment (start 104.7 121.2) (end 103.9 122) (width 0.3) (layer "F.Cu") (net 4))
-  (segment (start 101.8 122) (end 101.3 121.5) (width 0.3) (layer "F.Cu") (net 4))
+  (segment (start 101.3 83.01) (end 103.045 81.265) (width 0.3) (layer "F.Cu") (net 4))
   (segment (start 114.3 125.3) (end 114.3 109.5) (width 0.3) (layer "F.Cu") (net 4))
   (segment (start 124.7 102.5) (end 130.8 102.5) (width 0.3) (layer "F.Cu") (net 4))
+  (segment (start 106.6 107.9) (end 105.7 107.9) (width 0.3) (layer "F.Cu") (net 4))
   (segment (start 134.4 98.9) (end 134.4 95.5) (width 0.3) (layer "F.Cu") (net 4))
-  (segment (start 101.635 81.265) (end 108.5 81.265) (width 0.3) (layer "F.Cu") (net 4))
   (segment (start 126.9 116) (end 126.43 116.47) (width 0.3) (layer "F.Cu") (net 4))
   (segment (start 106.4 87.6) (end 106.4 93.48) (width 0.3) (layer "F.Cu") (net 4))
   (segment (start 106.4 93.48) (end 108.5 95.58) (width 0.3) (layer "F.Cu") (net 4))
-  (segment (start 108.5 106) (end 106.6 107.9) (width 0.3) (layer "F.Cu") (net 4))
   (segment (start 121 121.9) (end 121 125) (width 0.3) (layer "F.Cu") (net 4))
   (segment (start 132 116) (end 126.9 116) (width 0.3) (layer "F.Cu") (net 4))
-  (segment (start 106.6 107.9) (end 105.7 107.9) (width 0.3) (layer "F.Cu") (net 4))
+  (segment (start 105.7 107.9) (end 104.7 108.9) (width 0.3) (layer "F.Cu") (net 4))
   (segment (start 130.8 102.5) (end 134.4 98.9) (width 0.3) (layer "F.Cu") (net 4))
+  (segment (start 108.5 106) (end 106.6 107.9) (width 0.3) (layer "F.Cu") (net 4))
+  (segment (start 103.045 81.265) (end 108.5 81.265) (width 0.3) (layer "F.Cu") (net 4))
+  (segment (start 104.7 108.9) (end 104.7 121.2) (width 0.3) (layer "F.Cu") (net 4))
   (segment (start 133.9 95) (end 133.885 95.015) (width 0.3) (layer "F.Cu") (net 4))
+  (segment (start 104.7 121.2) (end 103.9 122) (width 0.3) (layer "F.Cu") (net 4))
   (segment (start 126.43 116.47) (end 121 121.9) (width 0.3) (layer "F.Cu") (net 4))
-  (segment (start 104.7 108.9) (end 104.7 121.2) (width 0.3) (layer "F.Cu") (net 4))
   (segment (start 133.885 95.015) (end 131.5 95.015) (width 0.3) (layer "F.Cu") (net 4))
   (segment (start 114.3 109.5) (end 116.135 107.665) (width 0.3) (layer "F.Cu") (net 4))
