File: ProyFinalMateriales/ProyFinalMateriales.kicad_sch (KiCad schematic)
At the start: 12 parts, among them U1 NodeMCU1.0(ESP-12E)

Commit message: update
Parts:
- removed BoostConverter1, Emisor1: Conn_01x03_Male, Connector_PinHeader_2.54mm:PinHeader_1x03_P2.54mm_Vertical, symbol Connector:Conn_01x03_Male
- removed Electromagnet1, SWITCH1: Conn_01x02_Male, Connector_PinHeader_2.54mm:PinHeader_1x02_P2.54mm_Vertical, symbol Connector:Conn_01x02_Male
- removed Receptor1: Conn_01x04_Male, Connector_PinHeader_2.54mm:PinHeader_1x04_P2.54mm_Vertical, symbol Connector:Conn_01x04_Male
Connections:
- net 3.3V1: now also TempHumd1.2 (Pin_2); no longer LED1.4 (Pin_4)
- net 3.3V3: now also LED1.4 (Pin_4); no longer TempHumd1.2 (Pin_2)
- net GND1: now also SensorPresion1.1 (Pin_1); no longer SensorPresion1.3 (Pin_3)
- net GPIO0: now also LED1.3 (Pin_3)
- net GPIO4: now also SensorPresion1.2 (Pin_2); no longer SensorPresion1.1 (Pin_1)
- net GPIO5: now also SensorPresion1.3 (Pin_3); no longer SensorPresion1.2 (Pin_2)
- net GPIO16: no longer names the net of U1.30 (D0(GPIO16))
